Commit message: Update diffbot.ros2_control.xacro

File: diffdrive_arduino-humble/description/ros2_control/diffbot.ros2_control.xacro (robot description, xacro)
@@ -1,5 +1,5 @@
 <?xml version="1.0"?>
 <robot xmlns:xacro="http://www.ros.org/wiki/xacro">
-  <xacro:macro name="diffbot_ros2_control" params="name prefix">
+  <!-- <xacro:macro name="diffbot_ros2_control" params="name prefix">
     <ros2_control name="${name}" type="system">
       <hardware>
@@ -28,4 +28,32 @@
       </joint>
     </ros2_control>
-  </xacro:macro>
+  </xacro:macro> -->
+  <ros2_control name="RealRobot" type="system">
+    <hardware>
+        <plugin>diffdrive_arduino/DiffDriveArduino</plugin>
+        <param name="left_wheel_name">left_wheel_joint</param>
+        <param name="right_wheel_name">right_wheel_joint</param>
+        <param name="loop_rate">30</param>
+        <param name="device">/dev/ttyUSB0</param>
+        <param name="baud_rate">57600</param>
+        <param name="timeout">1000</param>
+        <param name="enc_counts_per_rev">3450</param>
+    </hardware>
+<joint name="left_wheel_joint">
+    <command_interface name="velocity">
+        <param name="min">-10</param>
+        <param name="max">10</param>
+    </command_interface>
+    <state_interface name="position"></state_interface>
+    <state_interface name="velocity"></state_interface>
+</joint>
+<joint name="right_wheel_joint">
+    <command_interface name="velocity">
+        <param name="min">-10</param>
+        <param name="max">10</param>
+    </command_interface>
+    <state_interface name="position"></state_interface>
+    <state_interface name="velocity"></state_interface>
+</joint>
+  </ros2_control>
 </robot>

Commit message: Update diffbot.ros2_control.xacro

File: diffdrive_arduino-humble/description/ros2_control/diffbot.ros2_control.xacro (robot description, xacro)
@@ -29,4 +29,6 @@
     </ros2_control>
   </xacro:macro> -->
+  <xacro:macro name="diffbot_ros2_control" params="name prefix">
+  </xacro:macro>
   <ros2_control name="RealRobot" type="system">
     <hardware>
@@ -57,3 +59,4 @@
 </joint>
   </ros2_control>
+</xacro:macro>
 </robot>

Commit message: Update diffbot.ros2_control.xacro

File: diffdrive_arduino-humble/description/ros2_control/diffbot.ros2_control.xacro (robot description, xacro)
@@ -30,5 +30,4 @@
   </xacro:macro> -->
   <xacro:macro name="diffbot_ros2_control" params="name prefix">
-  </xacro:macro>
   <ros2_control name="RealRobot" type="system">
     <hardware>
@@ -42,20 +41,20 @@
         <param name="enc_counts_per_rev">3450</param>
     </hardware>
-<joint name="left_wheel_joint">
-    <command_interface name="velocity">
-        <param name="min">-10</param>
-        <param name="max">10</param>
-    </command_interface>
-    <state_interface name="position"></state_interface>
-    <state_interface name="velocity"></state_interface>
-</joint>
-<joint name="right_wheel_joint">
-    <command_interface name="velocity">
-        <param name="min">-10</param>
-        <param name="max">10</param>
-    </command_interface>
-    <state_interface name="position"></state_interface>
-    <state_interface name="velocity"></state_interface>
-</joint>
+    <joint name="left_wheel_joint">
+        <command_interface name="velocity">
+            <param name="min">-10</param>
+            <param name="max">10</param>
+        </command_interface>
+        <state_interface name="position"></state_interface>
+        <state_interface name="velocity"></state_interface>
+    </joint>
+    <joint name="right_wheel_joint">
+        <command_interface name="velocity">
+            <param name="min">-10</param>
+            <param name="max">10</param>
+        </command_interface>
+        <state_interface name="position"></state_interface>
+        <state_interface name="velocity"></state_interface>
+    </joint>
   </ros2_control>
 </xacro:macro>

Commit message: Update diffbot.ros2_control.xacro

File: diffdrive_arduino-humble/description/ros2_control/diffbot.ros2_control.xacro (robot description, xacro)
@@ -45,19 +45,13 @@
         <param name="pid_o">50</param>
     </hardware>
-    <joint name="left_wheel_joint">
-        <command_interface name="velocity">
-            <param name="min">-10</param>
-            <param name="max">10</param>
-        </command_interface>
-        <state_interface name="position"></state_interface>
-        <state_interface name="velocity"></state_interface>
+    <joint name="${prefix}left_wheel_joint">
+      <command_interface name="velocity"/>
+      <state_interface name="position"/>
+      <state_interface name="velocity"/>
     </joint>
-    <joint name="right_wheel_joint">
-        <command_interface name="velocity">
-            <param name="min">-10</param>
-            <param name="max">10</param>
-        </command_interface>
-        <state_interface name="position"></state_interface>
-        <state_interface name="velocity"></state_interface>
+    <joint name="${prefix}right_wheel_joint">
+      <command_interface name="velocity"/>
+      <state_interface name="position"/>
+      <state_interface name="velocity"/>
     </joint>
   </ros2_control>

Commit message: Update diffbot.ros2_control.xacro

File: diffdrive_arduino-humble/description/ros2_control/diffbot.ros2_control.xacro (robot description, xacro)
@@ -1,5 +1,5 @@
 <?xml version="1.0"?>
 <robot xmlns:xacro="http://www.ros.org/wiki/xacro">
-  <!-- <xacro:macro name="diffbot_ros2_control" params="name prefix">
+  <xacro:macro name="diffbot_ros2_control" params="name prefix">
     <ros2_control name="${name}" type="system">
       <hardware>
@@ -8,5 +8,5 @@
         <param name="right_wheel_name">right_wheel_joint</param>
         <param name="loop_rate">30</param>
-        <param name="device">/dev/serial/by-path/platform-fd500000.pcie-pci-0000:01:00.0-usb-0:1.3:1.0-port0</param>
+        <param name="device">/dev/ttyUSB0</param>
         <param name="baud_rate">57600</param>
         <param name="timeout_ms">1000</param>
@@ -28,6 +28,6 @@
       </joint>
     </ros2_control>
-  </xacro:macro> -->
-  <xacro:macro name="diffbot_ros2_control" params="name prefix">
+  </xacro:macro>
+  <!-- <xacro:macro name="diffbot_ros2_control" params="name prefix">
   <ros2_control name="RealRobot" type="system">
     <hardware>
@@ -56,4 +56,4 @@
     </joint>
   </ros2_control>
-</xacro:macro>
+</xacro:macro> -->
 </robot>
